Commit message: added the robot_bringup package and  bs_bringup package
basic functionality for debugging all hardware, all sensors are supported,

-controller in the next version

File: robot_v1_description/urdf/robot_core.xacro (robot description, xacro)
@@ -13,4 +13,7 @@
     <material name="black">
         <color rgba="0 0 0 1"/>
+    </material>
+    <material name="red">
+        <color rgba="1 0 0 1"/>
     </material>
     <!-- BASE LINK -->
@@ -92,5 +95,5 @@
         <parent link="chassis"/>
         <child link="caster_wheel_front"/>
-        <origin xyz="0.38 0 0"/>
+        <origin xyz="0.34 0 0"/>
     </joint>
     <link name="caster_wheel_front">
@@ -133,3 +136,4 @@
     </link>
     <!-- SENSORS -->
+    <xacro:include filename="sensors.xacro" />
 </robot>
